File: key_matrix.sch (KiCad schematic (older format))
At the start: 190 parts

Commit message: Schematic & Footprint bindings
Parts:
- D1, D10, D11, D12, D13, D14, D15, D16, D17, D18, D19, D2, D20, D21, D22, D23, D24, D25, D26, D27, D28, D29, D3, D30, D31, D32, D33, D34, D35, D36, D37, D38, D39, D4, D40, D41, D42, D43, D44, D45, D46, D47, D48, D49, D5, D50, D51, D52, D53, D54, D55, D56, D57, D58, D59, D6, D60, D61, D62, D63, D64, D65, D66, D67, D68, D69, D7, D70, D71, D72, D73, D74, D75, D76, D77, D78, D79, D8, D80, D81, D82, D83, D84, D85, D86, D87, D88, D89, D9, D90, D91, D92, D93, D94, D95: renamed from D?; footprint (none) -> Diode_SMD:D_SOD-123
- MX0-0, MX0-1, MX0-10, MX0-11, MX0-12, MX0-13, MX0-14, MX0-15, MX0-16, MX0-17, MX0-2, MX0-3, MX0-4, MX0-5, MX0-6, MX0-7, MX0-8, MX0-9, MX1-0, MX1-1, MX1-10, MX1-11, MX1-12, MX1-13, MX1-14, MX1-17, MX1-2, MX1-3, MX1-4, MX1-5, MX1-6, MX1-7, MX1-8, MX1-9, MX2-0, MX2-1, MX2-10, MX2-11, MX2-12, MX2-13, MX2-14, MX2-17, MX2-3, MX2-4, MX2-5, MX2-6, MX2-7, MX2-8, MX2-9, MX3-0, MX3-1, MX3-10, MX3-11, MX3-12, MX3-13, MX3-17, MX3-3, MX3-4, MX3-5, MX3-6, MX3-7, MX3-8, MX3-9, MX4-0, MX4-1, MX4-10, MX4-11, MX4-12, MX4-16, MX4-17, MX4-3, MX4-4, MX4-5, MX4-6, MX4-7, MX4-8, MX4-9, MX5-0, MX5-1, MX5-13, MX5-16, MX5-17, MX5-3: value MX-LED -> MX-NoLED; footprint (none) -> MX_Only:MXOnly-1U-NoLED; symbol MX_Alps_Hybrid:MX-LED -> MX_Alps_Hybrid:MX-NoLED
- MX1-16: value MX-LED -> MX-NoLED; footprint (none) -> MX_Only:MXOnly-2U-NoLED; symbol MX_Alps_Hybrid:MX-LED -> MX_Alps_Hybrid:MX-NoLED
- MX2-16, MX2-2, MX5-11, MX5-12, MX5-2, MX5-4: value MX-LED -> MX-NoLED; footprint (none) -> MX_Only:MXOnly-1.5U-NoLED; symbol MX_Alps_Hybrid:MX-LED -> MX_Alps_Hybrid:MX-NoLED
- MX3-16, MX4-2: value MX-LED -> MX-NoLED; footprint (none) -> MX_Only:MXOnly-2.25U-NoLED; symbol MX_Alps_Hybrid:MX-LED -> MX_Alps_Hybrid:MX-NoLED
- MX3-2, MX4-13: value MX-LED -> MX-NoLED; footprint (none) -> MX_Only:MXOnly-1.75U-NoLED; symbol MX_Alps_Hybrid:MX-LED -> MX_Alps_Hybrid:MX-NoLED
- MX5-8: value MX-LED -> MX-NoLED; footprint (none) -> MX_Only:MXOnly-6U-Centered-NoLED; symbol MX_Alps_Hybrid:MX-LED -> MX_Alps_Hybrid:MX-NoLED

Commit message: Routing & LEDS
Parts:
- MX5-11: footprint MX_Only:MXOnly-1.5U-NoLED -> MX_Only:MXOnly-1.25U-NoLED
- MX5-8: footprint MX_Only:MXOnly-6U-Centered-NoLED -> MX_Only:MXOnly-6.25U-NoLED
Connections:
- net ROW4: now also D18.1 (K)
Other:
- moved on the sheet: D18, MX4-2
Changed lines of the file:
@@
 $Descr A4 11693 8268
 encoding utf-8
-Sheet 2 2
+Sheet 2 3
 Title ""
 Date ""
@@
 Wire Wire Line
 	1700 4000 1850 4000
-$Comp
-L MX_Alps_Hybrid:MX-NoLED MX?
-U 1 1 5DA4DDFA
-P 2600 3900
-AR Path="/5DA4DDFA" Ref="MX?"  Part="1"
-AR Path="/5D9B08E9/5DA4DDFA" Ref="MX4-2"  Part="1"
-F 0 "MX4-2" H 2682 4124 60  0000 C CNN
-F 1 "MX-NoLED" H 2682 4050 20  0000 C CNN
-F 2 "MX_Only:MXOnly-2.25U-NoLED" H 1975 3875 60  0001 C CNN
-F 3 "" H 1975 3875 60  0001 C CNN
-	1    2600 3900
-	1    0    0    -1
-$EndComp
-$Comp
-L Device:D_Small D18
-U 1 1 5DA4DE00
-P 2400 4150
-F 0 "D18" V 2446 4082 50  0000 R CNN
-F 1 "SOD-123" V 2355 4082 50  0000 R CNN
-F 2 "Diode_SMD:D_SOD-123" V 2400 4150 50  0001 C CNN
-F 3 "~" V 2400 4150 50  0001 C CNN
-	1    2400 4150
-	0    -1   -1   0
-$EndComp
 Wire Wire Line
-	2400 4050 2550 4050
+	2400 4000 2550 4000
 $Comp
 L MX_Alps_Hybrid:MX-NoLED MX?
@@
 F 0 "MX5-8" H 6032 4674 60  0000 C CNN
 F 1 "MX-NoLED" H 6032 4600 20  0000 C CNN
-F 2 "MX_Only:MXOnly-6U-Centered-NoLED" H 5325 4425 60  0001 C CNN
+F 2 "MX_Only:MXOnly-6.25U-NoLED" H 5325 4425 60  0001 C CNN
 F 3 "" H 5325 4425 60  0001 C CNN
 	1    5950 4450
@@
 F 0 "MX5-11" H 7982 4674 60  0000 C CNN
 F 1 "MX-NoLED" H 7982 4600 20  0000 C CNN
-F 2 "MX_Only:MXOnly-1.5U-NoLED" H 7275 4425 60  0001 C CNN
+F 2 "MX_Only:MXOnly-1.25U-NoLED" H 7275 4425 60  0001 C CNN
 F 3 "" H 7275 4425 60  0001 C CNN
 	1    7900 4450
@@
 Connection ~ 10300 3800
 Wire Wire Line
-	2750 3850 2750 4400
-Wire Wire Line
 	2750 4400 2650 4400
-Wire Wire Line
-	2750 3200 2750 3850
 Connection ~ 2750 3200
-Connection ~ 2750 3850
 Wire Wire Line
 	3450 3200 3450 3700
@@
 	1150 4200 1700 4200
 Connection ~ 1700 4200
-Wire Wire Line
-	1700 4200 3300 4200
 Connection ~ 3300 4200
 Wire Wire Line
@@
 Connection ~ 4800 1400
 Connection ~ 4800 2000
+Wire Wire Line
+	1700 4200 2400 4200
+Wire Wire Line
+	2750 3200 2750 3800
+$Comp
+L MX_Alps_Hybrid:MX-NoLED MX?
+U 1 1 5DA4DDFA
+P 2600 3850
+AR Path="/5DA4DDFA" Ref="MX?"  Part="1"
+AR Path="/5D9B08E9/5DA4DDFA" Ref="MX4-2"  Part="1"
+F 0 "MX4-2" H 2682 4074 60  0000 C CNN
+F 1 "MX-NoLED" H 2682 4000 20  0000 C CNN
+F 2 "MX_Only:MXOnly-2.25U-NoLED" H 1975 3825 60  0001 C CNN
+F 3 "" H 1975 3825 60  0001 C CNN
+	1    2600 3850
+	1    0    0    -1
+$EndComp
+$Comp
+L Device:D_Small D18
+U 1 1 5DA4DE00
+P 2400 4100
+F 0 "D18" V 2446 4032 50  0000 R CNN
+F 1 "SOD-123" V 2355 4032 50  0000 R CNN
+F 2 "Diode_SMD:D_SOD-123" V 2400 4100 50  0001 C CNN
+F 3 "~" V 2400 4100 50  0001 C CNN
+	1    2400 4100
+	0    -1   -1   0
+$EndComp
+Connection ~ 2400 4200
+Wire Wire Line
+	2400 4200 3300 4200
+Connection ~ 2750 3800
+Wire Wire Line
+	2750 3800 2750 4400
 $EndSCHEMATC
